File: Hardware/Helgatchi back PCB/Helgatchi back PCB.kicad_sch (KiCad schematic)
At the start: 8 parts, among them J1 u.FL, J2 RP-SMA

Commit message: Drawings and laser cutter files
Parts:
- H1, H2: footprint MountingHole:MountingHole_2.2mm_M2_Pad_Via -> MountingHole:MountingHole_2.2mm_M2_Pad
- J2: footprint Connector_Coaxial:SMA_Samtec_SMA-J-P-H-ST-EM1_EdgeMount -> Connector_Coaxial:SMA_Amphenol_901-143_Horizontal; LCSC Part # (none) -> C1509217
Changed lines of the file:
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@@
 			)
 		)
-		(property "Footprint" "MountingHole:MountingHole_2.2mm_M2_Pad_Via"
+		(property "Footprint" "MountingHole:MountingHole_2.2mm_M2_Pad"
 			(at 127 96.52 0)
 			(effects
@@
 			)
 		)
-		(property "Footprint" "MountingHole:MountingHole_2.2mm_M2_Pad_Via"
+		(property "Footprint" "MountingHole:MountingHole_2.2mm_M2_Pad"
 			(at 114.3 96.52 0)
 			(effects
@@
 			)
 		)
-		(property "Footprint" "Connector_Coaxial:SMA_Samtec_SMA-J-P-H-ST-EM1_EdgeMount"
+		(property "Footprint" "Connector_Coaxial:SMA_Amphenol_901-143_Horizontal"
 			(at 91.44 95.25 0)
 			(effects
@@
 			)
 		)
-		(property "LCSC Part #" ""
+		(property "LCSC Part #" "C1509217"
 			(at 91.44 95.25 0)
 			(effects

Commit message: Update back PCB to R2.7
Parts:
- H1, H2: footprint MountingHole:MountingHole_2.2mm_M2_Pad -> MountingHole:MountingHole_2.2mm_M2_Pad_Via
- H3, H4, H5, H6: footprint Sinhoo SMTSO 2M:SMTSO M2 solder pad -> MountingHole:MountingHole_2.2mm_M2_Pad_Via
- J1: LCSC Part # (none) -> C411563
Changed lines of the file:
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@@
 			)
 		)
-		(property "Footprint" "Sinhoo SMTSO 2M:SMTSO M2 solder pad"
+		(property "Footprint" "MountingHole:MountingHole_2.2mm_M2_Pad_Via"
 			(at 175.26 96.52 0)
 			(effects
@@
 			)
 		)
-		(property "Footprint" "MountingHole:MountingHole_2.2mm_M2_Pad"
+		(property "Footprint" "MountingHole:MountingHole_2.2mm_M2_Pad_Via"
 			(at 127 96.52 0)
 			(effects
@@
 			)
 		)
-		(property "Footprint" "MountingHole:MountingHole_2.2mm_M2_Pad"
+		(property "Footprint" "MountingHole:MountingHole_2.2mm_M2_Pad_Via"
 			(at 114.3 96.52 0)
 			(effects
@@
 			)
 		)
-		(property "Footprint" "Sinhoo SMTSO 2M:SMTSO M2 solder pad"
+		(property "Footprint" "MountingHole:MountingHole_2.2mm_M2_Pad_Via"
 			(at 193.04 96.52 0)
 			(effects
@@
 			)
 		)
-		(property "Footprint" "Sinhoo SMTSO 2M:SMTSO M2 solder pad"
+		(property "Footprint" "MountingHole:MountingHole_2.2mm_M2_Pad_Via"
 			(at 157.48 96.52 0)
 			(effects
@@
 			)
 		)
-		(property "Footprint" "Sinhoo SMTSO 2M:SMTSO M2 solder pad"
+		(property "Footprint" "MountingHole:MountingHole_2.2mm_M2_Pad_Via"
 			(at 210.82 96.52 0)
 			(effects
@@
 			)
 		)
-		(property "LCSC Part #" ""
+		(property "LCSC Part #" "C411563"
 			(at 78.74 95.25 0)
 			(effects
