File: Hardware/Helgatchi front PCB/Helgatchi front PCB.kicad_pcb (KiCad board)
At the start: 2 copper layers, 50 x 80 mm, 39 parts, among them J1 BATTERY, J2 SCREEN, M1 MOTOR, Q1 NMOS, SW1 LEFT BUTTON, SW2 CENTER BUTTON, SW3 RIGHT BUTTON, U1 XIAO ESP32-S3

Commit message: Start of R2.8
- Moving to SK6805s for LEDs
- imported footprint, symbol, and 3D model for SK6805-SIDE
- updated footprints and symbols for LEDs
- repositioned LEDs and capacitors
- Swapped LED chain direction to accommodate easier routing with new pinout
Parts:
- D2, D3, D4, D5, D6, D7: value WS2812C-4020-H2 -> SK6805-SIDE; footprint WS2812:WS2812C-4020-H2 -> SK68XX-SIDE:LED-SMD_4P-L3.5-W1.6_SK6805SIDE-G-001
- moved D3 41.5 mm to (181.0, 76.5)
- moved D2 33.5 mm to (181.0, 121.0)
- moved D5 33.5 mm to (147.0, 76.5)
- moved D7 33.5 mm to (147.0, 121.0)
- moved C7 26.6 mm to (181.0, 93.0), turned to 180 degrees
- moved D4 24.0 mm to (147.0, 100.5), turned to 90 degrees
- moved C2 3.81 mm to (148.5, 100.5), turned to 90 degrees
- moved C1 3.35 mm to (148.5, 121.0), turned to 90 degrees
- moved C3 3.35 mm to (148.5, 76.5), turned to 90 degrees
- moved D6 0.71 mm to (181.0, 100.5), turned to -90 degrees
Connections:
- D2 pad 1: LED_CONTROL -> Net-(D2-DOUT)
- D2 pad 2: +3.3V -> GND
- D2 pad 3: Net-(D2-DOUT) -> +3.3V
- D2 pad 4: GND -> LED_CONTROL
- D3 pad 1: Net-(D2-DOUT) -> Net-(D3-DOUT)
- D3 pad 2: +3.3V -> GND
- D3 pad 3: Net-(D3-DOUT) -> +3.3V
- D3 pad 4: GND -> Net-(D2-DOUT)
- D4 pad 1: Net-(D3-DOUT) -> Net-(D4-DOUT)
- D4 pad 2: +3.3V -> GND
- D4 pad 3: Net-(D4-DOUT) -> +3.3V
- D4 pad 4: GND -> Net-(D3-DOUT)
- D5 pad 1: Net-(D4-DOUT) -> Net-(D5-DOUT)
- D5 pad 2: +3.3V -> GND
- D5 pad 3: Net-(D5-DOUT) -> +3.3V
- D5 pad 4: GND -> Net-(D4-DOUT)
- D6 pad 1: Net-(D5-DOUT) -> Net-(D6-DOUT)
- D6 pad 2: +3.3V -> GND
- D6 pad 3: Net-(D6-DOUT) -> +3.3V
- D6 pad 4: GND -> Net-(D5-DOUT)
- D7 pad 1: Net-(D6-DOUT) -> unconnected-(D7-DOUT-Pad1)
- D7 pad 2: +3.3V -> GND
- D7 pad 3: unconnected-(D7-DOUT-Pad3) -> +3.3V
- D7 pad 4: GND -> Net-(D6-DOUT)
Routing:
- net +3.3V: track 289.2 -> 97.9 mm
- net Net-(D4-DOUT): track 50.3 -> 0.00 mm
- net Net-(D5-DOUT): track 24.5 -> 0.00 mm
- net Net-(D3-DOUT): track 24.4 -> 0.00 mm
- net Net-(D6-DOUT): track 19.7 -> 0.00 mm
- net Net-(D2-DOUT): track 19.7 -> 0.00 mm
- net LED_CONTROL: track 15.9 -> 0.00 mm
- net GND: vias 39 -> 33
Other:
- board text added: "${REVISION}-${CURRENT_DATE} ${}"
- board text removed: "HW-${REVISION}-${CURRENT_DATE} ${}"

Commit message: Wrap up R2.8
Boards ordered, version locked
Parts:
- moved D4 41.6 mm to (181.0, 76.5), turned to -90 degrees
- moved C7 38.0 mm to (175.0, 130.5), turned to -90 degrees
- moved D6 34.0 mm to (147.0, 100.5), turned to 90 degrees
- moved D3 24.0 mm to (181.0, 100.5)
- moved C4 3.35 mm to (179.5, 76.5), turned to -90 degrees
- moved C6 3.35 mm to (179.5, 121.0), turned to -90 degrees
- moved C5 2.92 mm to (179.5, 100.5), turned to -90 degrees
- moved J1 0.25 mm to (176.5, 125.5)
Routing:
- net +3.3V: track 97.9 -> 189.7 mm, vias 4 -> 9
- net Net-(D4-DOUT): track 0.00 -> 48.3 mm
- net LED_CONTROL: track 0.00 -> 37.2 mm
- net Net-(D5-DOUT): track 0.00 -> 22.2 mm
- net Net-(D3-DOUT): track 0.00 -> 22.2 mm
- net GND: track 27.3 -> 46.3 mm, vias 33 -> 34
- net Net-(D6-DOUT): track 0.00 -> 17.8 mm
- net Net-(D2-DOUT): track 0.00 -> 17.2 mm
Other:
- board text added: "HELLO THERE!"

Commit message: Commit new UI files
Parts:
- added TP1: BATT, TestPoint:TestPoint_Pad_D1.0mm, B.Cu at (181.0, 125.5)
Routing:
- net +BATT: track 38.7 -> 42.7 mm
- net LED_CONTROL: track 37.2 -> 38.4 mm

Commit message: final R2.9 revision, boards ordered
Parts:
- removed C7: 10uF, Capacitor_SMD:C_0603_1608Metric
- added REF**: Fiducial_0.5mm_Mask2mm, Fiducial:Fiducial_0.5mm_Mask2mm, B.Cu at (174.0, 62.5)
- added REF**: Fiducial_0.5mm_Mask2mm, Fiducial:Fiducial_0.5mm_Mask2mm, B.Cu at (151.0, 135.5)
- added REF**: Fiducial_0.5mm_Mask2mm, Fiducial:Fiducial_0.5mm_Mask2mm, B.Cu at (177.0, 135.5)
- added REF**: Fiducial_0.5mm_Mask2mm, Fiducial:Fiducial_0.5mm_Mask2mm, B.Cu at (154.0, 62.5)
Connections:
- C1 pad 2: +3.3V -> +BATT
- C2 pad 2: +3.3V -> +BATT
- C3 pad 2: +3.3V -> +BATT
- C4 pad 2: +3.3V -> +BATT
- C5 pad 2: +3.3V -> +BATT
- C6 pad 2: +3.3V -> +BATT
- D1 pad 1: +3.3V -> +BATT
- D2 pad 3: +3.3V -> +BATT
- D3 pad 3: +3.3V -> +BATT
- D4 pad 3: +3.3V -> +BATT
- D5 pad 3: +3.3V -> +BATT
- D6 pad 3: +3.3V -> +BATT
- D7 pad 3: +3.3V -> +BATT
- M1 pad 1: +3.3V -> +BATT
Routing:
- net +BATT: track 42.7 -> 233.2 mm, vias 0 -> 3
- net +3.3V: track 189.7 -> 43.3 mm, vias 9 -> 2
- net GND: track 46.3 -> 44.1 mm, vias 34 -> 39
